Commit message: xacro macros seperated

File: xacro/barista_robot_model.urdf.xacro (robot description, xacro)
@@ -1,274 +1,4 @@
 <?xml version="1.0"?>
 <robot xmlns:xacro="http://www.ros.org/wiki/xacro" name="barista_robot">
-<material name="red">
-    <color rgba="1.0 0.0 0.0 1"/>
-</material>
-<material name="green_light">
-    <color rgba="0.0 1.0 0.0 1"/>
-</material>
-<material name="green_dark">
-<color rgba="0.0 0.5 0.0 1"/>
-</material>
-<material name="blue">
-    <color rgba="0.0 0.0 1.0 1"/>
-</material>
-<material name="black">
-    <color rgba="0.1 0.1 0.1 1"/>
-</material>
-<material name="grey">
-    <color rgba="0.5 0.5 0.5 1"/>
-</material>
-<xacro:macro name="drive_wheel" params="side parent xyz">
-  <joint name="joint_${side}_wheel" type="continuous">
-    <origin rpy="0 0 0" xyz="${xyz}"/>
-    <parent link="${parent}"/>
-    <child link="${side}_wheel"/>
-    <axis xyz="0 1 0"/>
-  </joint>
-  <link name="${side}_wheel">
-    <visual>
-      <origin rpy="0 1.5707 1.5707"/>
-      <geometry>
-        <cylinder length="0.0206" radius="0.0352"/>
-      </geometry>
-      <material name="black"/>
-    </visual>
-    <collision>
-      <origin rpy="0 1.5707 1.5707"/>
-      <geometry>
-        <cylinder length="0.0206" radius="0.0352"/>
-      </geometry>
-    </collision>
-    <inertial>
-      <mass value="1.0"/>
-      <origin xyz="0 0 0" rpy="0 1.5707 1.5707"/>
-      <inertia ixx="0.00061952" ixy="0" ixz="0" iyy="0.00013216" iyz="0" izz="0.00013216"/>
-    </inertial>
-  </link>
-  <gazebo reference="${side}_wheel">
-    <kp>1000000000000000000000000000.0</kp>
-    <kd>1000000000000000000000000000.0</kd>
-    <mu1>1.0</mu1>
-    <mu2>1.0</mu2>
-    <material>Gazebo/Black</material>
-  </gazebo>
-</xacro:macro>
-<xacro:macro name="caster_wheel" params="parent xyz">
-  <!-- caster_yaw_joint -->
-  <joint name="caster_yaw_joint" type="continuous">
-    <origin rpy="0 0 0" xyz="${xyz}"/>
-    <parent link="${parent}"/>
-    <child link="caster_yaw_link"/>
-    <axis xyz="0 0 1"/>
-    <limit effort="1000.0" velocity="100.0" />
-    <dynamics damping="0.0" friction="0.1"/>
-  </joint>
-  <link name="caster_yaw_link">
-    <visual>
-      <origin rpy="0 1.5707 1.5707" xyz="0 0 0"/>
-      <geometry>
-        <cylinder length="0.001" radius="0.0352"/>
-      </geometry>
-      <material name="blue"/>
-    </visual>
-    <collision>
-      <origin rpy="0 1.5707 1.5707" xyz="0 0 0"/>
-      <geometry>
-        <cylinder length="0.001" radius="0.0352"/>
-      </geometry>
-    </collision>
-    <inertial>
-        <origin rpy="0 1.5707 1.5707" xyz="0 0 0"/>
-        <mass value="0.05"/>
-        <inertia ixx="5.175e-05" ixy="0.0" ixz="0.0" iyy="5.175e-05" iyz="0.0" izz="3.097e-05"/>
-    </inertial>
-  </link>
-  <!-- caster_roll_joint -->
-  <joint name="caster_roll_joint" type="continuous">
-    <origin xyz="0 0 0" rpy="0 0 0"/>
-    <parent link="caster_yaw_link"/>
-    <child link="caster_roll_link"/>
-    <axis xyz="1 0 0"/>
-    <limit effort="1000.0" velocity="100.0" />
-    <dynamics damping="0.0" friction="0.1"/>
-  </joint>
-  <link name="caster_roll_link">
-    <visual>
-      <origin rpy="0 1.5707 1.5707" xyz="0 0 0"/>
-      <geometry>
-        <cylinder length="0.001" radius="0.0352"/>
-      </geometry>
-      <material name="red"/>
-    </visual>
-    <collision>
-      <origin rpy="0 1.5707 1.5707" xyz="0 0 0"/>
-      <geometry>
-        <cylinder length="0.001" radius="0.0352"/>
-      </geometry>
-    </collision>
-    <inertial>
-        <origin rpy="0 1.5707 1.5707" xyz="0 0 0"/>
-        <mass value="0.05"/>
-        <inertia ixx="5.175e-05" ixy="0.0" ixz="0.0" iyy="5.175e-05" iyz="0.0" izz="3.097e-05"/>
-    </inertial>
-  </link>
-  <!-- caster_pitch_joint -->
-  <joint name="caster_pitch_joint" type="continuous">
-    <origin xyz="0 0 0" rpy="0 0 0"/>
-    <parent link="caster_roll_link"/>
-    <child link="caster_pitch_link"/>
-    <axis xyz="0 1 0"/>
-    <limit effort="1000.0" velocity="100.0" />
-    <dynamics damping="0.0" friction="0.1"/>
-  </joint>
-  <link name="caster_pitch_link">
-    <visual>
-      <origin rpy="0 1.5707 1.5707" xyz="0 0 0"/>
-      <geometry>
-        <sphere radius="0.0352"/>
-      </geometry>
-      <material name="green_dark"/>
-    </visual>
-    <collision>
-      <origin rpy="0 1.5707 1.5707" xyz="0 0 0"/>
-      <geometry>
-        <sphere radius="0.0352"/>
-      </geometry>
-    </collision>
-    <inertial>
-        <origin rpy="0 1.5707 1.5707" xyz="0 0 0"/>
-        <mass value="1."/>
-        <inertia ixx="0.0004952" ixy="0.0" ixz="0.0" iyy="0.0004952" iyz="0.0" izz="0.0004952"/>
-    </inertial>
-  </link>
-  <gazebo reference="caster_pitch_link">
-    <kp>1000000000000000000000000000.0</kp>
-    <kd>1000000000000000000000000000.0</kd>
-    <mu1>1.0</mu1>
-    <mu2>1.0</mu2>
-    <material>Gazebo/Green</material>
-  </gazebo>
-</xacro:macro>
-<xacro:macro name="standoff_rod" params="name parent xyz length radius">
-  <joint name="${name}_joint" type="fixed">
-    <origin rpy="0 0 0" xyz="${xyz}"/>
-    <parent link="${parent}"/>
-    <child link="${name}"/>
-  </joint>
-  <link name="${name}">
-    <visual>
-      <geometry>
-        <cylinder length="${length}" radius="${radius}"/>
-      </geometry>
-      <material name="grey"/>
-    </visual>
-    <collision>
-      <geometry>
-        <cylinder length="${length}" radius="${radius}"/>
-      </geometry>
-    </collision>
-    <inertial>
-      <mass value="0.3"/>
-      <origin rpy="0 0 0" xyz="0 0 0"/>
-      <inertia ixx="0.00121675" ixy="0" ixz="0" iyy="0.00121675" iyz="0" izz="0.000015"/>
-    </inertial>
-  </link>
-  <gazebo reference="${name}">
-    <kp>1000000000000000000000000000.0</kp>
-    <kd>1000000000000000000000000000.0</kd>
-    <mu1>1.0</mu1>
-    <mu2>1.0</mu2>
-    <material>Gazebo/Grey</material>
-  </gazebo>
-</xacro:macro>
-<xacro:macro name="cup_holder_tray" params="parent xyz">
-  <joint name="cupholder_tray_joint" type="fixed">
-    <origin rpy="0 0 0" xyz="${xyz}"/>
-    <parent link="${parent}"/>
-    <child link="cupholder_tray"/>
-  </joint>
-  <link name="cupholder_tray">
-    <visual>
-      <geometry>
-        <cylinder length="0.09" radius="0.16"/>
-      </geometry>
-      <material name="blue"/>
-    </visual>
-    <collision>
-      <geometry>
-        <cylinder length="0.09" radius="0.16"/>
-      </geometry>
-    </collision>
-    <inertial>
-      <mass value="5.0"/>
-      <origin rpy="0 0 0" xyz="0 0 0"/>
-      <inertia ixx="0.0102" ixy="0" ixz="0" iyy="0.0102" iyz="0" izz="0.064"/>
-    </inertial>
-  </link>
-  <gazebo reference="cupholder_tray">
-    <kp>1000000000000000000000000000.0</kp>
-    <kd>1000000000000000000000000000.0</kd>
-    <mu1>1.0</mu1>
-    <mu2>1.0</mu2>
-    <material>Gazebo/Blue</material>
-  </gazebo>
-</xacro:macro>
-<xacro:macro name="laser_scanner" params="parent xyz">
-  <joint name="joint_laser_scan" type="fixed">
-    <origin rpy="0 0 0" xyz="${xyz}"/>
-    <parent link="${parent}"/>
-    <child link="laser_scan_link"/>
-  </joint>
-  <link name="laser_scan_link">
-    <visual>
-       <origin rpy="0 0 0" xyz="0 0 -0.055"/>
-      <geometry>
-        <mesh filename="package://barista_robot_description/meshes/sensors/hokuyo_urg_04lx.dae" scale="1.0 1.0 1.0"/>
-      </geometry>
-    </visual>
-    <collision>
-       <origin rpy="0 0 0" xyz="0 0 -0.055"/>
-      <geometry>
-        <box size="0.06 0.06 0.08"/>
-      </geometry>
-    </collision>
-    <inertial>
-      <mass value="0.05"/>
-      <origin rpy="0 0 0" xyz="0 0 -0.055"/>
-      <inertia ixx="1.067e-05" ixy="0" ixz="0" iyy="6.0e-06" iyz="0" izz="1.067e-05"/>
-    </inertial>
-  </link>
-  <gazebo reference="laser_scan_link">
-      <sensor name="sensor_ray" type="ray">
-          <pose>0 0 0 0 0 0</pose>
-          <ray>
-            <scan>
-              <horizontal>
-                <samples>1024</samples>
-                <resolution>1.0</resolution>
-                <min_angle>-3.14</min_angle>
-                <max_angle>3.14</max_angle>
-              </horizontal>
-            </scan>
-            <range>
-              <min>0.02</min>
-              <max>5.6</max>
-            </range>
-          </ray>
-          <always_on>true</always_on>
-          <visualize>true</visualize>
-          <update_rate>100.0</update_rate>
-          <plugin name="laser" filename="libgazebo_ros_ray_sensor.so">
-            <ros>
-              <namespace>/barista_robot</namespace>
-              <remapping>~/out:=laser_scan</remapping>
-            </ros>
-            <output_type>sensor_msgs/LaserScan</output_type>
-            <frame_name>laser_scan_link</frame_name>
-          </plugin>
-      </sensor>
-  </gazebo>
-</xacro:macro>
-<!--
   <xacro:include filename="$(find barista_robot_description)/xacro/drive_wheel.xacro"/>
   <xacro:include filename="$(find barista_robot_description)/xacro/caster_wheel.xacro"/>
@@ -276,5 +6,5 @@
   <xacro:include filename="$(find barista_robot_description)/xacro/cup_holder_tray.xacro"/>
   <xacro:include filename="$(find barista_robot_description)/xacro/laser_scanner.xacro"/>
- -->
+  <xacro:include filename="$(find barista_robot_description)/xacro/barista_robot.gazebo.xacro" />
   <xacro:property name="include_laser" value="true"/>
   <link name="base_link">
@@ -290,5 +20,7 @@
           <cylinder length="0.155" radius="0.178"/>
       </geometry>
-      <material name="blue"/>
+      <material name="Gazebo/Blue">
+          <color rgba="0.0 0.0 1.0 1.0"/>
+      </material>
     </visual>
     <collision>
@@ -303,57 +35,21 @@
     </inertial>
   </link>
-  <gazebo reference="chassis">
-    <kp>1000000000000000000000000000.0</kp>
-    <kd>1000000000000000000000000000.0</kd>
-    <mu1>1.0</mu1>
-    <mu2>1.0</mu2>
-    <material>Gazebo/Blue</material>
-  </gazebo>
-  <!-- Drive wheels -->
+  <!-- Drive wheels macro -->
   <xacro:drive_wheel side="left" parent="chassis" xyz="-0.05 0.13 -0.078"/>
   <xacro:drive_wheel side="right" parent="chassis" xyz="-0.05 -0.13 -0.078"/>
-  <!-- Caster wheel -->
+  <!-- Caster wheel macro -->
   <xacro:caster_wheel parent="chassis" xyz="0.13 0 -0.078"/>
-  <!-- Standoff rods -->
-  <xacro:standoff_rod name="standoff_rod_left" parent="chassis" xyz="0 0.12 0.188" length="0.22" radius="0.01"/>
-  <xacro:standoff_rod name="standoff_rod_right" parent="chassis" xyz="0 -0.12 0.188" length="0.22" radius="0.01"/>
-  <!-- Cup holder tray -->
+  <!-- Standoff rods macro -->
+  <xacro:standoff_rod name="standoff_rod_fl" parent="chassis" xyz="0.03 0.13 0.188" length="0.22" radius="0.01"/>
+  <xacro:standoff_rod name="standoff_rod_fr" parent="chassis" xyz="0.03 -0.13 0.188" length="0.22" radius="0.01"/>
+  <xacro:standoff_rod name="standoff_rod_bl" parent="chassis" xyz="-0.03 0.13 0.188" length="0.22" radius="0.01"/>
+  <xacro:standoff_rod name="standoff_rod_br" parent="chassis" xyz="-0.03 -0.13 0.188" length="0.22" radius="0.01"/>
+  <!-- Cup holder tray macro -->
   <xacro:cup_holder_tray parent="chassis" xyz="0 0.0 0.343"/>
-  <!-- Conditionally include laser -->
+  <!-- Conditionally include laser macro -->
   <xacro:if value="${include_laser}">
     <xacro:laser_scanner parent="chassis" xyz="0.11 0 0.1325"/>
   </xacro:if>
-  <!-- JOINT PUBLISHER -->
-  <gazebo>
-    <plugin name="barista_joint_state" filename="libgazebo_ros_joint_state_publisher.so">
-      <ros>
-          <remapping>~/out:=joint_states</remapping>
-      </ros>
-      <update_rate>30</update_rate>
-      <joint_name>joint_left_wheel</joint_name>
-      <joint_name>joint_right_wheel</joint_name>
-      <joint_name>caster_yaw_joint</joint_name>
-      <joint_name>caster_roll_joint</joint_name>
-      <joint_name>caster_pitch_joint</joint_name>
-    </plugin>
-  </gazebo>
-  <!-- Differential drive -->
-  <gazebo>
-    <plugin filename="libgazebo_ros_diff_drive.so" name="differential_drive_controller">
-      <!-- wheels -->
-      <left_joint>joint_left_wheel</left_joint>
-      <right_joint>joint_right_wheel</right_joint>
-      <!-- kinematics -->
-      <wheel_separation>0.26</wheel_separation>
-      <wheel_diameter>0.07</wheel_diameter>
-      <!-- limits -->
-      <max_wheel_torque>1.0</max_wheel_torque>
-      <max_wheel_acceleration>2.0</max_wheel_acceleration>
-      <!-- output -->
-      <publish_odom>true</publish_odom>
-      <publish_odom_tf>true</publish_odom_tf>
-      <odometry_frame>odom</odometry_frame>
-      <robot_base_frame>base_link</robot_base_frame>
-    </plugin>
-  </gazebo>
+  <!-- Gazebo elements macro -->
+  <xacro:gazebo_elements/>
 </robot>
