Commit message: spawned two robots

File: xacro/barista_robot.gazebo.xacro (robot description, xacro)
@@ -8,5 +8,5 @@
     <mu1>1.0</mu1>
     <mu2>1.0</mu2>
-    <material>Gazebo/Blue</material>
+    <material>${robot_color_gz}</material>
   </gazebo>
   <gazebo reference="cupholder_tray">
@@ -15,5 +15,5 @@
     <mu1>1.0</mu1>
     <mu2>1.0</mu2>
-    <material>Gazebo/Blue</material>
+    <material>${robot_color_gz}</material>
   </gazebo>
   <gazebo reference="standoff_rod_fl">
@@ -68,6 +68,7 @@
   <!-- Joint State Publisher -->
   <gazebo>
-    <plugin name="barista_joint_state" filename="libgazebo_ros_joint_state_publisher.so">
+    <plugin name="${robot_name}_joint_state" filename="libgazebo_ros_joint_state_publisher.so">
       <ros>
+          <namespace>${robot_name}</namespace>
           <remapping>~/out:=joint_states</remapping>
       </ros>
@@ -82,5 +83,8 @@
   <!-- Differential drive -->
   <gazebo>
-    <plugin filename="libgazebo_ros_diff_drive.so" name="differential_drive_controller">
+    <plugin name="${robot_name}_differential_drive_controller" filename="libgazebo_ros_diff_drive.so">
+      <ros>
+          <namespace>${robot_name}</namespace>
+      </ros>
       <!-- wheels -->
       <left_joint>joint_left_wheel</left_joint>
@@ -95,6 +99,6 @@
       <publish_odom>true</publish_odom>
       <publish_odom_tf>true</publish_odom_tf>
-      <odometry_frame>odom</odometry_frame>
-      <robot_base_frame>base_link</robot_base_frame>
+      <odometry_frame>${robot_name}/odom</odometry_frame>
+      <robot_base_frame>${robot_name}/base_link</robot_base_frame>
     </plugin>
   </gazebo>
@@ -120,11 +124,11 @@
           <visualize>true</visualize>
           <update_rate>100.0</update_rate>
-          <plugin name="laser" filename="libgazebo_ros_ray_sensor.so">
+          <plugin name="${robot_name}_laser" filename="libgazebo_ros_ray_sensor.so">
             <ros>
-              <!-- <namespace>/</namespace> -->
+              <namespace>${robot_name}</namespace>
               <remapping>~/out:=/scan</remapping>
             </ros>
             <output_type>sensor_msgs/LaserScan</output_type>
-            <frame_name>laser_scan_link</frame_name>
+            <frame_name>${robot_name}/laser_scan_link</frame_name>
           </plugin>
       </sensor>

File: xacro/barista_robot_model.urdf.xacro (robot description, xacro)
@@ -1,4 +1,6 @@
 <?xml version="1.0"?>
-<robot xmlns:xacro="http://www.ros.org/wiki/xacro" name="barista_robot">
+<robot xmlns:xacro="http://www.ros.org/wiki/xacro" robot_namespace="" name="barista_robot">
+  <xacro:property name="robot_name" value="$(arg robot_name)"/>
+  <xacro:property name="include_laser" value="true"/>
   <xacro:include filename="$(find barista_robot_description)/xacro/drive_wheel.xacro"/>
   <xacro:include filename="$(find barista_robot_description)/xacro/caster_wheel.xacro"/>
@@ -7,5 +9,14 @@
   <xacro:include filename="$(find barista_robot_description)/xacro/laser_scanner.xacro"/>
   <xacro:include filename="$(find barista_robot_description)/xacro/barista_robot.gazebo.xacro" />
-  <xacro:property name="include_laser" value="true"/>
+  <!-- Robot color macro -->
+  <xacro:if value="${robot_name == 'rick'}">
+    <xacro:property name="robot_color_gz" value="Gazebo/Red"/>
+    <xacro:property name="robot_color" value="1.0 0.0 0.0 1.0"/>
+  </xacro:if>
+  <xacro:unless value="${robot_name == 'rick'}">
+    <xacro:property name="robot_color_gz" value="Gazebo/Blue"/>
+    <xacro:property name="robot_color" value="0.0 0.0 1.0 1.0"/>
+  </xacro:unless>
+  <!-- Robot chassis -->
   <link name="base_link">
   </link>
@@ -20,6 +31,6 @@
           <cylinder length="0.155" radius="0.178"/>
       </geometry>
-      <material name="Gazebo/Blue">
-          <color rgba="0.0 0.0 1.0 1.0"/>
+      <material name="Robot Color">
+          <color rgba="${robot_color}"/>
       </material>
     </visual>
@@ -52,4 +63,4 @@
   </xacro:if>
   <!-- Gazebo elements macro -->
-  <xacro:gazebo_elements/>
+  <xacro:gazebo_elements />
 </robot>

File: xacro/cup_holder_tray.xacro (robot description, xacro)
@@ -12,6 +12,6 @@
         <cylinder length="0.09" radius="0.16"/>
       </geometry>
-      <material name="Gazebo/Blue">
-          <color rgba="0.0 0.0 1.0 1.0"/>
+      <material name="Robot Color">
+          <color rgba="${robot_color}"/>
       </material>
     </visual>

Commit message: added prefix to all robot links and joints

File: xacro/barista_robot.gazebo.xacro (robot description, xacro)
@@ -3,5 +3,5 @@
 <xacro:macro name="gazebo_elements">
   <!-- Robot Elements -->
-  <gazebo reference="chassis">
+  <gazebo reference="${prefix}chassis">
     <kp>1000000000000000000000000000.0</kp>
     <kd>1000000000000000000000000000.0</kd>
@@ -10,5 +10,5 @@
     <material>${robot_color_gz}</material>
   </gazebo>
-  <gazebo reference="cupholder_tray">
+  <gazebo reference="${prefix}cupholder_tray">
     <kp>1000000000000000000000000000.0</kp>
     <kd>1000000000000000000000000000.0</kd>
@@ -17,5 +17,5 @@
     <material>${robot_color_gz}</material>
   </gazebo>
-  <gazebo reference="standoff_rod_fl">
+  <gazebo reference="${prefix}standoff_rod_fl">
     <kp>1000000000000000000000000000.0</kp>
     <kd>1000000000000000000000000000.0</kd>
@@ -24,5 +24,5 @@
     <material>Gazebo/Grey</material>
   </gazebo>
-  <gazebo reference="standoff_rod_fr">
+  <gazebo reference="${prefix}standoff_rod_fr">
     <kp>1000000000000000000000000000.0</kp>
     <kd>1000000000000000000000000000.0</kd>
@@ -31,5 +31,5 @@
     <material>Gazebo/Grey</material>
   </gazebo>
-  <gazebo reference="standoff_rod_bl">
+  <gazebo reference="${prefix}standoff_rod_bl">
     <kp>1000000000000000000000000000.0</kp>
     <kd>1000000000000000000000000000.0</kd>
@@ -38,5 +38,5 @@
     <material>Gazebo/Grey</material>
   </gazebo>
-  <gazebo reference="standoff_rod_br">
+  <gazebo reference="${prefix}standoff_rod_br">
     <kp>1000000000000000000000000000.0</kp>
     <kd>1000000000000000000000000000.0</kd>
@@ -45,5 +45,5 @@
     <material>Gazebo/Grey</material>
   </gazebo>
-  <gazebo reference="left_wheel">
+  <gazebo reference="${prefix}left_wheel">
     <kp>1000000000000000000000000000.0</kp>
     <kd>1000000000000000000000000000.0</kd>
@@ -52,5 +52,5 @@
     <material>Gazebo/Black</material>
   </gazebo>
-  <gazebo reference="right_wheel">
+  <gazebo reference="${prefix}right_wheel">
     <kp>1000000000000000000000000000.0</kp>
     <kd>1000000000000000000000000000.0</kd>
@@ -59,5 +59,5 @@
     <material>Gazebo/Black</material>
   </gazebo>
-  <gazebo reference="caster_pitch_link">
+  <gazebo reference="${prefix}caster_pitch_link">
     <kp>1000000000000000000000000000.0</kp>
     <kd>1000000000000000000000000000.0</kd>
@@ -70,13 +70,13 @@
     <plugin name="${robot_name}_joint_state" filename="libgazebo_ros_joint_state_publisher.so">
       <ros>
-          <namespace>${robot_name}</namespace>
+          <namespace>/${robot_name}</namespace>
           <remapping>~/out:=joint_states</remapping>
       </ros>
       <update_rate>30</update_rate>
-      <joint_name>joint_left_wheel</joint_name>
-      <joint_name>joint_right_wheel</joint_name>
-      <joint_name>caster_yaw_joint</joint_name>
-      <joint_name>caster_roll_joint</joint_name>
-      <joint_name>caster_pitch_joint</joint_name>
+      <joint_name>${prefix}joint_left_wheel</joint_name>
+      <joint_name>${prefix}joint_right_wheel</joint_name>
+      <joint_name>${prefix}caster_yaw_joint</joint_name>
+      <joint_name>${prefix}caster_roll_joint</joint_name>
+      <joint_name>${prefix}caster_pitch_joint</joint_name>
     </plugin>
   </gazebo>
@@ -85,24 +85,20 @@
     <plugin name="${robot_name}_differential_drive_controller" filename="libgazebo_ros_diff_drive.so">
       <ros>
-          <namespace>${robot_name}</namespace>
+          <namespace>/${robot_name}</namespace>
       </ros>
-      <!-- wheels -->
-      <left_joint>joint_left_wheel</left_joint>
-      <right_joint>joint_right_wheel</right_joint>
-      <!-- kinematics -->
+      <left_joint>${prefix}joint_left_wheel</left_joint>
+      <right_joint>${prefix}joint_right_wheel</right_joint>
       <wheel_separation>0.26</wheel_separation>
       <wheel_diameter>0.07</wheel_diameter>
-      <!-- limits -->
       <max_wheel_torque>1.0</max_wheel_torque>
       <max_wheel_acceleration>2.0</max_wheel_acceleration>
-      <!-- output -->
       <publish_odom>true</publish_odom>
       <publish_odom_tf>true</publish_odom_tf>
-      <odometry_frame>${robot_name}/odom</odometry_frame>
-      <robot_base_frame>${robot_name}/base_link</robot_base_frame>
+      <odometry_frame>${prefix}odom</odometry_frame>
+      <robot_base_frame>${prefix}base_link</robot_base_frame>
     </plugin>
   </gazebo>
   <!-- Lidar plugin -->
-  <gazebo reference="laser_scan_link">
+  <gazebo reference="${prefix}laser_scan_link">
       <sensor name="sensor_ray" type="ray">
           <pose>0 0 0 0 0 0</pose>
@@ -126,9 +122,9 @@
           <plugin name="${robot_name}_laser" filename="libgazebo_ros_ray_sensor.so">
             <ros>
-              <namespace>${robot_name}</namespace>
-              <remapping>~/out:=/scan</remapping>
+              <namespace>/${robot_name}</namespace>
+              <remapping>~/out:=/${prefix}scan</remapping>
             </ros>
             <output_type>sensor_msgs/LaserScan</output_type>
-            <frame_name>${robot_name}/laser_scan_link</frame_name>
+            <frame_name>${prefix}laser_scan_link</frame_name>
           </plugin>
       </sensor>

File: xacro/barista_robot_model.urdf.xacro (robot description, xacro)
@@ -1,5 +1,6 @@
 <?xml version="1.0"?>
-<robot xmlns:xacro="http://www.ros.org/wiki/xacro" robot_namespace="" name="barista_robot">
+<robot xmlns:xacro="http://www.ros.org/wiki/xacro" name="barista_robot">
   <xacro:property name="robot_name" value="$(arg robot_name)"/>
+  <xacro:property name="prefix" value="$(arg robot_name)/"/>
   <xacro:property name="include_laser" value="true"/>
   <xacro:include filename="$(find barista_robot_description)/xacro/drive_wheel.xacro"/>
@@ -19,12 +20,12 @@
   </xacro:unless>
   <!-- Robot chassis -->
-  <link name="base_link">
+  <link name="${prefix}base_link">
   </link>
-  <joint name="base_link_joint" type="fixed">
+  <joint name="${prefix}base_link_joint" type="fixed">
     <origin rpy="0 0 0" xyz="0 0 0.1132" />
-    <parent link="base_link" />
-    <child link="chassis" />
+    <parent link="${prefix}base_link" />
+    <child link="${prefix}chassis" />
   </joint>
-  <link name="chassis">
+  <link name="${prefix}chassis">
     <visual>
       <geometry>
@@ -47,20 +48,20 @@
   </link>
   <!-- Drive wheels macro -->
-  <xacro:drive_wheel side="left" parent="chassis" xyz="-0.05 0.13 -0.078"/>
-  <xacro:drive_wheel side="right" parent="chassis" xyz="-0.05 -0.13 -0.078"/>
+  <xacro:drive_wheel side="left" parent="${prefix}chassis" xyz="-0.05 0.13 -0.078"/>
+  <xacro:drive_wheel side="right" parent="${prefix}chassis" xyz="-0.05 -0.13 -0.078"/>
   <!-- Caster wheel macro -->
-  <xacro:caster_wheel parent="chassis" xyz="0.13 0 -0.078"/>
+  <xacro:caster_wheel parent="${prefix}chassis" xyz="0.13 0 -0.078"/>
   <!-- Standoff rods macro -->
-  <xacro:standoff_rod name="standoff_rod_fl" parent="chassis" xyz="0.03 0.13 0.188" length="0.22" radius="0.01"/>
-  <xacro:standoff_rod name="standoff_rod_fr" parent="chassis" xyz="0.03 -0.13 0.188" length="0.22" radius="0.01"/>
-  <xacro:standoff_rod name="standoff_rod_bl" parent="chassis" xyz="-0.03 0.13 0.188" length="0.22" radius="0.01"/>
-  <xacro:standoff_rod name="standoff_rod_br" parent="chassis" xyz="-0.03 -0.13 0.188" length="0.22" radius="0.01"/>
+  <xacro:standoff_rod name="${prefix}standoff_rod_fl" parent="${prefix}chassis" xyz="0.03 0.13 0.188" length="0.22" radius="0.01"/>
+  <xacro:standoff_rod name="${prefix}standoff_rod_fr" parent="${prefix}chassis" xyz="0.03 -0.13 0.188" length="0.22" radius="0.01"/>
+  <xacro:standoff_rod name="${prefix}standoff_rod_bl" parent="${prefix}chassis" xyz="-0.03 0.13 0.188" length="0.22" radius="0.01"/>
+  <xacro:standoff_rod name="${prefix}standoff_rod_br" parent="${prefix}chassis" xyz="-0.03 -0.13 0.188" length="0.22" radius="0.01"/>
   <!-- Cup holder tray macro -->
-  <xacro:cup_holder_tray parent="chassis" xyz="0 0.0 0.343"/>
+  <xacro:cup_holder_tray parent="${prefix}chassis" xyz="0 0.0 0.343"/>
   <!-- Conditionally include laser macro -->
   <xacro:if value="${include_laser}">
-    <xacro:laser_scanner parent="chassis" xyz="0.11 0 0.1325"/>
+    <xacro:laser_scanner parent="${prefix}chassis" xyz="0.11 0 0.1325"/>
   </xacro:if>
-  <!-- Gazebo elements macro -->
+  <!-- Gazebo elements/plugins macro -->
   <xacro:gazebo_elements />
 </robot>

File: xacro/caster_wheel.xacro (robot description, xacro)
@@ -3,13 +3,13 @@
 <xacro:macro name="caster_wheel" params="parent xyz">
   <!-- caster_yaw_joint -->
-  <joint name="caster_yaw_joint" type="continuous">
+  <joint name="${prefix}caster_yaw_joint" type="continuous">
     <origin rpy="0 0 0" xyz="${xyz}"/>
     <parent link="${parent}"/>
-    <child link="caster_yaw_link"/>
+    <child link="${prefix}caster_yaw_link"/>
     <axis xyz="0 0 1"/>
     <limit effort="1000.0" velocity="100.0" />
     <dynamics damping="0.0" friction="0.1"/>
   </joint>
-  <link name="caster_yaw_link">
+  <link name="${prefix}caster_yaw_link">
     <visual>
       <origin rpy="0 1.5707 1.5707" xyz="0 0 0"/>
@@ -34,13 +34,13 @@
   </link>
   <!-- caster_roll_joint -->
-  <joint name="caster_roll_joint" type="continuous">
+  <joint name="${prefix}caster_roll_joint" type="continuous">
     <origin xyz="0 0 0" rpy="0 0 0"/>
-    <parent link="caster_yaw_link"/>
-    <child link="caster_roll_link"/>
+    <parent link="${prefix}caster_yaw_link"/>
+    <child link="${prefix}caster_roll_link"/>
     <axis xyz="1 0 0"/>
     <limit effort="1000.0" velocity="100.0" />
     <dynamics damping="0.0" friction="0.1"/>
   </joint>
-  <link name="caster_roll_link">
+  <link name="${prefix}caster_roll_link">
     <visual>
       <origin rpy="0 1.5707 1.5707" xyz="0 0 0"/>
@@ -65,13 +65,13 @@
   </link>
   <!-- caster_pitch_joint -->
-  <joint name="caster_pitch_joint" type="continuous">
+  <joint name="${prefix}caster_pitch_joint" type="continuous">
     <origin xyz="0 0 0" rpy="0 0 0"/>
-    <parent link="caster_roll_link"/>
-    <child link="caster_pitch_link"/>
+    <parent link="${prefix}caster_roll_link"/>
+    <child link="${prefix}caster_pitch_link"/>
     <axis xyz="0 1 0"/>
     <limit effort="1000.0" velocity="100.0" />
     <dynamics damping="0.0" friction="0.1"/>
   </joint>
-  <link name="caster_pitch_link">
+  <link name="${prefix}caster_pitch_link">
     <visual>
       <origin rpy="0 1.5707 1.5707" xyz="0 0 0"/>

File: xacro/cup_holder_tray.xacro (robot description, xacro)
@@ -2,10 +2,10 @@
 <robot xmlns:xacro="http://www.ros.org/wiki/xacro">
 <xacro:macro name="cup_holder_tray" params="parent xyz">
-  <joint name="cupholder_tray_joint" type="fixed">
+  <joint name="${prefix}cupholder_tray_joint" type="fixed">
     <origin rpy="0 0 0" xyz="${xyz}"/>
     <parent link="${parent}"/>
-    <child link="cupholder_tray"/>
+    <child link="${prefix}cupholder_tray"/>
   </joint>
-  <link name="cupholder_tray">
+  <link name="${prefix}cupholder_tray">
     <visual>
       <geometry>

File: xacro/drive_wheel.xacro (robot description, xacro)
@@ -2,11 +2,11 @@
 <robot xmlns:xacro="http://www.ros.org/wiki/xacro">
 <xacro:macro name="drive_wheel" params="side parent xyz">
-  <joint name="joint_${side}_wheel" type="continuous">
+  <joint name="${prefix}joint_${side}_wheel" type="continuous">
     <origin rpy="0 0 0" xyz="${xyz}"/>
     <parent link="${parent}"/>
-    <child link="${side}_wheel"/>
+    <child link="${prefix}${side}_wheel"/>
     <axis xyz="0 1 0"/>
   </joint>
-  <link name="${side}_wheel">
+  <link name="${prefix}${side}_wheel">
     <visual>
       <origin rpy="0 1.5707 1.5707"/>

File: xacro/laser_scanner.xacro (robot description, xacro)
@@ -2,10 +2,10 @@
 <robot xmlns:xacro="http://www.ros.org/wiki/xacro">
 <xacro:macro name="laser_scanner" params="parent xyz">
-  <joint name="joint_laser_scan" type="fixed">
+  <joint name="${prefix}joint_laser_scan" type="fixed">
     <origin rpy="0 0 0" xyz="${xyz}"/>
     <parent link="${parent}"/>
-    <child link="laser_scan_link"/>
+    <child link="${prefix}laser_scan_link"/>
   </joint>
-  <link name="laser_scan_link">
+  <link name="${prefix}laser_scan_link">
     <visual>
        <origin rpy="0 0 0" xyz="0 0 -0.055"/>

Commit message: added back caster wheel - rviz view adjusted to chase

File: xacro/barista_robot.gazebo.xacro (robot description, xacro)
@@ -59,5 +59,12 @@
     <material>Gazebo/Black</material>
   </gazebo>
-  <gazebo reference="${prefix}caster_pitch_link">
+  <gazebo reference="${prefix}front_caster_pitch_link">
+    <kp>1000000000000000000000000000.0</kp>
+    <kd>1000000000000000000000000000.0</kd>
+    <mu1>1.0</mu1>
+    <mu2>1.0</mu2>
+    <material>Gazebo/Green</material>
+  </gazebo>
+  <gazebo reference="${prefix}back_caster_pitch_link">
     <kp>1000000000000000000000000000.0</kp>
     <kd>1000000000000000000000000000.0</kd>
@@ -76,7 +83,10 @@
       <joint_name>${prefix}joint_left_wheel</joint_name>
       <joint_name>${prefix}joint_right_wheel</joint_name>
-      <joint_name>${prefix}caster_yaw_joint</joint_name>
-      <joint_name>${prefix}caster_roll_joint</joint_name>
-      <joint_name>${prefix}caster_pitch_joint</joint_name>
+      <joint_name>${prefix}front_caster_yaw_joint</joint_name>
+      <joint_name>${prefix}front_caster_roll_joint</joint_name>
+      <joint_name>${prefix}front_caster_pitch_joint</joint_name>
+      <joint_name>${prefix}back_caster_yaw_joint</joint_name>
+      <joint_name>${prefix}back_caster_roll_joint</joint_name>
+      <joint_name>${prefix}back_caster_pitch_joint</joint_name>
     </plugin>
   </gazebo>

File: xacro/barista_robot_model.urdf.xacro (robot description, xacro)
@@ -15,8 +15,8 @@
     <xacro:property name="robot_color" value="1.0 0.0 0.0 1.0"/>
   </xacro:if>
-  <xacro:unless value="${robot_name == 'rick'}">
+  <xacro:if value="${robot_name == 'morty'}">
     <xacro:property name="robot_color_gz" value="Gazebo/Blue"/>
     <xacro:property name="robot_color" value="0.0 0.0 1.0 1.0"/>
-  </xacro:unless>
+  </xacro:if>
   <!-- Robot chassis -->
   <link name="${prefix}base_link">
@@ -48,8 +48,9 @@
   </link>
   <!-- Drive wheels macro -->
-  <xacro:drive_wheel side="left" parent="${prefix}chassis" xyz="-0.05 0.13 -0.078"/>
-  <xacro:drive_wheel side="right" parent="${prefix}chassis" xyz="-0.05 -0.13 -0.078"/>
+  <xacro:drive_wheel side="left" parent="${prefix}chassis" xyz="0.0 0.14 -0.078"/>
+  <xacro:drive_wheel side="right" parent="${prefix}chassis" xyz="0.0 -0.14 -0.078"/>
   <!-- Caster wheel macro -->
-  <xacro:caster_wheel parent="${prefix}chassis" xyz="0.13 0 -0.078"/>
+  <xacro:caster_wheel side="front" parent="${prefix}chassis" xyz="0.13 0 -0.078"/>
+  <xacro:caster_wheel side="back" parent="${prefix}chassis" xyz="-0.13 0 -0.078"/>
   <!-- Standoff rods macro -->
   <xacro:standoff_rod name="${prefix}standoff_rod_fl" parent="${prefix}chassis" xyz="0.03 0.13 0.188" length="0.22" radius="0.01"/>

File: xacro/caster_wheel.xacro (robot description, xacro)
@@ -1,15 +1,15 @@
 <?xml version="1.0"?>
 <robot xmlns:xacro="http://www.ros.org/wiki/xacro">
-<xacro:macro name="caster_wheel" params="parent xyz">
+<xacro:macro name="caster_wheel" params="side parent xyz">
   <!-- caster_yaw_joint -->
-  <joint name="${prefix}caster_yaw_joint" type="continuous">
+  <joint name="${prefix}${side}_caster_yaw_joint" type="continuous">
     <origin rpy="0 0 0" xyz="${xyz}"/>
     <parent link="${parent}"/>
-    <child link="${prefix}caster_yaw_link"/>
+    <child link="${prefix}${side}_caster_yaw_link"/>
     <axis xyz="0 0 1"/>
     <limit effort="1000.0" velocity="100.0" />
     <dynamics damping="0.0" friction="0.1"/>
   </joint>
-  <link name="${prefix}caster_yaw_link">
+  <link name="${prefix}${side}_caster_yaw_link">
     <visual>
       <origin rpy="0 1.5707 1.5707" xyz="0 0 0"/>
@@ -34,13 +34,13 @@
   </link>
   <!-- caster_roll_joint -->
-  <joint name="${prefix}caster_roll_joint" type="continuous">
+  <joint name="${prefix}${side}_caster_roll_joint" type="continuous">
     <origin xyz="0 0 0" rpy="0 0 0"/>
-    <parent link="${prefix}caster_yaw_link"/>
-    <child link="${prefix}caster_roll_link"/>
+    <parent link="${prefix}${side}_caster_yaw_link"/>
+    <child link="${prefix}${side}_caster_roll_link"/>
     <axis xyz="1 0 0"/>
     <limit effort="1000.0" velocity="100.0" />
     <dynamics damping="0.0" friction="0.1"/>
   </joint>
-  <link name="${prefix}caster_roll_link">
+  <link name="${prefix}${side}_caster_roll_link">
     <visual>
       <origin rpy="0 1.5707 1.5707" xyz="0 0 0"/>
@@ -65,13 +65,13 @@
   </link>
   <!-- caster_pitch_joint -->
-  <joint name="${prefix}caster_pitch_joint" type="continuous">
+  <joint name="${prefix}${side}_caster_pitch_joint" type="continuous">
     <origin xyz="0 0 0" rpy="0 0 0"/>
-    <parent link="${prefix}caster_roll_link"/>
-    <child link="${prefix}caster_pitch_link"/>
+    <parent link="${prefix}${side}_caster_roll_link"/>
+    <child link="${prefix}${side}_caster_pitch_link"/>
     <axis xyz="0 1 0"/>
     <limit effort="1000.0" velocity="100.0" />
     <dynamics damping="0.0" friction="0.1"/>
   </joint>
-  <link name="${prefix}caster_pitch_link">
+  <link name="${prefix}${side}_caster_pitch_link">
     <visual>
       <origin rpy="0 1.5707 1.5707" xyz="0 0 0"/>
